File: 1999_Dodge_Dakota.kicad_sch (KiCad schematic)
At the start: 13 parts, among them J101 Conn_01x23, J102 Conn_01x35, J103 Conn_01x35, J105 Conn_01x01, J107 Conn_01x01, J108 Conn_01x01

Commit message: Draft breakout board check in.
Parts:
- added J11: Dodge_Con, Dodge_Cons:1999_Dodge_Connector_32x3cons, symbol 1999_Dodge_Connector_32x3cons:Dodge_Con
- added J?: Conn_02x32_Counter_Clockwise, symbol Connector_Generic:Conn_02x32_Counter_Clockwise
Other:
- moved on the sheet: C17, D101, D102, D103, D104, F101, F102, J101, J102, J103, J105, J107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
