File: lowside_quad.kicad_sch (KiCad schematic)
At the start: 4 parts, among them U201 VNLD5160, U202 VNLD5160

Commit message: File names changed / moved to folders. Updated file names to 1999_Dodge_Dakota Moved files footprints and symbols into a folder
Other:
- title: rusEfi Proteus -> 1999 Dodge Dakota Based on rusEFI/proteus
Changed lines of the file:
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@@
 (kicad_sch (version 20211123) (generator eeschema)
-  (paper "A4")
+  (paper "B")
   (title_block
-    (title "rusEfi Proteus")
-    (date "2022-04-09")
-    (rev "v0.7")
+    (title "1999 Dodge Dakota Based on rusEFI/proteus")
+    (date "2023-08-12")
+    (rev "V0.1")
     (company "rusEFI")
-    (comment 1 "github.com/mck1117/proteus")
-    (comment 2 "rusefi.com/s/proteus")
   )
   (junction (at 70.485 76.2) (diameter 0) (color 0 0 0 0)
