File: Breakout_1999_Dodge_Dakota.kicad_pcb (KiCad board)
At the start: 4 copper layers, 215 x 195 mm, 391 parts, among them J1 Dodge_Con, U1 ACS712xLCTR-20A

Commit message: Another draft check in. Deleted unused "export" files.
Parts:
- removed F385: Fuse_Holder, LCSC_parts:LCSC_C492610_Fuse_holder
- removed F386, F387, F388, F389: Pig_Con, TestPoint:TestPoint_THTPad_1.5x1.5mm_Drill0.7mm
- added F1193: Fuse_Holder, LCSC_parts:LCSC_C2935870_Fuse_holder, F.Cu at (222.5, 216.0)
- added F1194: Fuse_Holder, LCSC_parts:LCSC_C2935870_Fuse_holder, F.Cu at (203.0, 216.0)
- added F1195: Fuse_Holder, LCSC_parts:LCSC_C2935870_Fuse_holder, F.Cu at (184.5, 215.5)
- added F1196: Fuse_Holder, LCSC_parts:LCSC_C2935870_Fuse_holder, F.Cu at (220.5, 231.5)
- added F1197: Fuse_Holder, LCSC_parts:LCSC_C2935870_Fuse_holder, F.Cu at (203.0, 231.5)
- added F1198: Fuse_Holder, LCSC_parts:LCSC_C2935870_Fuse_holder, F.Cu at (185.5, 231.0)
- added F1385: Pig_Con, TestPoint:TestPoint_THTPad_1.5x1.5mm_Drill0.7mm, F.Cu at (217.6, 206.5)
- added F1386: Pig_Con, TestPoint:TestPoint_THTPad_1.5x1.5mm_Drill0.7mm, F.Cu at (198.1, 206.5)
- added F1387: Pig_Con, TestPoint:TestPoint_THTPad_1.5x1.5mm_Drill0.7mm, F.Cu at (217.6, 210.5)
- added F1389: Pig_Con, TestPoint:TestPoint_THTPad_1.5x1.5mm_Drill0.7mm, F.Cu at (197.6, 211.0)
- added F1391: Pig_Con, TestPoint:TestPoint_THTPad_1.5x1.5mm_Drill0.7mm, F.Cu at (227.6, 211.0)
- added F1392: Pig_Con, TestPoint:TestPoint_THTPad_1.5x1.5mm_Drill0.7mm, F.Cu at (208.1, 210.5)
- added F1393: Pig_Con, TestPoint:TestPoint_THTPad_1.5x1.5mm_Drill0.7mm, F.Cu at (227.6, 206.0)
- added F1394: Pig_Con, TestPoint:TestPoint_THTPad_1.5x1.5mm_Drill0.7mm, F.Cu at (207.6, 206.5)
- added F1395: Pig_Con, TestPoint:TestPoint_THTPad_1.5x1.5mm_Drill0.7mm, F.Cu at (179.6, 206.5)
- added F1396: Pig_Con, TestPoint:TestPoint_THTPad_1.5x1.5mm_Drill0.7mm, F.Cu at (216.1, 222.0)
- added F1397: Pig_Con, TestPoint:TestPoint_THTPad_1.5x1.5mm_Drill0.7mm, F.Cu at (179.6, 210.5)
- added F1399: Pig_Con, TestPoint:TestPoint_THTPad_1.5x1.5mm_Drill0.7mm, F.Cu at (216.1, 226.5)
- added F1401: Pig_Con, TestPoint:TestPoint_THTPad_1.5x1.5mm_Drill0.7mm, F.Cu at (189.6, 206.0)
- added F1402: Pig_Con, TestPoint:TestPoint_THTPad_1.5x1.5mm_Drill0.7mm, F.Cu at (225.6, 226.0)
- added F1403: Pig_Con, TestPoint:TestPoint_THTPad_1.5x1.5mm_Drill0.7mm, F.Cu at (189.6, 210.5)
- added F1404: Pig_Con, TestPoint:TestPoint_THTPad_1.5x1.5mm_Drill0.7mm, F.Cu at (225.6, 222.0)
- added F1405: Pig_Con, TestPoint:TestPoint_THTPad_1.5x1.5mm_Drill0.7mm, F.Cu at (198.6, 222.0)
- added F1406: Pig_Con, TestPoint:TestPoint_THTPad_1.5x1.5mm_Drill0.7mm, F.Cu at (180.6, 221.0)
- added F1407: Pig_Con, TestPoint:TestPoint_THTPad_1.5x1.5mm_Drill0.7mm, F.Cu at (198.6, 226.0)
- added F1409: Pig_Con, TestPoint:TestPoint_THTPad_1.5x1.5mm_Drill0.7mm, F.Cu at (180.6, 225.5)
- added F1411: Pig_Con, TestPoint:TestPoint_THTPad_1.5x1.5mm_Drill0.7mm, F.Cu at (208.6, 226.0)
- added F1412: Pig_Con, TestPoint:TestPoint_THTPad_1.5x1.5mm_Drill0.7mm, F.Cu at (190.6, 225.5)
- added F1413: Pig_Con, TestPoint:TestPoint_THTPad_1.5x1.5mm_Drill0.7mm, F.Cu at (208.1, 222.0)
- added F1414: Pig_Con, TestPoint:TestPoint_THTPad_1.5x1.5mm_Drill0.7mm, F.Cu at (190.6, 221.5)
- added U2: ACS712xLCTR-20A, Package_SO:SOIC-8_3.9x4.9mm_P1.27mm, F.Cu at (203.1, 209.0)
- added U3: ACS712xLCTR-20A, Package_SO:SOIC-8_3.9x4.9mm_P1.27mm, F.Cu at (184.6, 208.5)
- added U4: ACS712xLCTR-20A, Package_SO:SOIC-8_3.9x4.9mm_P1.27mm, F.Cu at (220.6, 224.5)
- added U5: ACS712xLCTR-20A, Package_SO:SOIC-8_3.9x4.9mm_P1.27mm, F.Cu at (203.1, 224.5)
- added U6: ACS712xLCTR-20A, Package_SO:SOIC-8_3.9x4.9mm_P1.27mm, F.Cu at (185.6, 224.0)
- F101: renamed from F1; footprint LCSC_parts:LCSC_C492610_Fuse_holder -> LCSC_parts:LCSC_C2935870_Fuse_holder
- F102: renamed from F2; footprint LCSC_parts:LCSC_C492610_Fuse_holder -> LCSC_parts:LCSC_C2935870_Fuse_holder
- F103: renamed from F3; footprint LCSC_parts:LCSC_C492610_Fuse_holder -> LCSC_parts:LCSC_C2935870_Fuse_holder
- F104: renamed from F4; footprint LCSC_parts:LCSC_C492610_Fuse_holder -> LCSC_parts:LCSC_C2935870_Fuse_holder
- F105: renamed from F5; footprint LCSC_parts:LCSC_C492610_Fuse_holder -> LCSC_parts:LCSC_C2935870_Fuse_holder
- F106: renamed from F6; footprint LCSC_parts:LCSC_C492610_Fuse_holder -> LCSC_parts:LCSC_C2935870_Fuse_holder
- F107: renamed from F7; footprint LCSC_parts:LCSC_C492610_Fuse_holder -> LCSC_parts:LCSC_C2935870_Fuse_holder
- F108: renamed from F8; footprint LCSC_parts:LCSC_C492610_Fuse_holder -> LCSC_parts:LCSC_C2935870_Fuse_holder
- F109: renamed from F9; footprint LCSC_parts:LCSC_C492610_Fuse_holder -> LCSC_parts:LCSC_C2935870_Fuse_holder
- F110: renamed from F10; footprint LCSC_parts:LCSC_C492610_Fuse_holder -> LCSC_parts:LCSC_C2935870_Fuse_holder
- F111: renamed from F11; footprint LCSC_parts:LCSC_C492610_Fuse_holder -> LCSC_parts:LCSC_C2935870_Fuse_holder
- F112: renamed from F34; footprint LCSC_parts:LCSC_C492610_Fuse_holder -> LCSC_parts:LCSC_C2935870_Fuse_holder
- F113: renamed from F35; footprint LCSC_parts:LCSC_C492610_Fuse_holder -> LCSC_parts:LCSC_C2935870_Fuse_holder
- F114: renamed from F36; footprint LCSC_parts:LCSC_C492610_Fuse_holder -> LCSC_parts:LCSC_C2935870_Fuse_holder
- F115: renamed from F37; footprint LCSC_parts:LCSC_C492610_Fuse_holder -> LCSC_parts:LCSC_C2935870_Fuse_holder
- F116: renamed from F38; footprint LCSC_parts:LCSC_C492610_Fuse_holder -> LCSC_parts:LCSC_C2935870_Fuse_holder
- F117: renamed from F39; footprint LCSC_parts:LCSC_C492610_Fuse_holder -> LCSC_parts:LCSC_C2935870_Fuse_holder
- F118: renamed from F40; footprint LCSC_parts:LCSC_C492610_Fuse_holder -> LCSC_parts:LCSC_C2935870_Fuse_holder
- F119: renamed from F41; footprint LCSC_parts:LCSC_C492610_Fuse_holder -> LCSC_parts:LCSC_C2935870_Fuse_holder
- F120: renamed from F42; footprint LCSC_parts:LCSC_C492610_Fuse_holder -> LCSC_parts:LCSC_C2935870_Fuse_holder
- F121: renamed from F43; footprint LCSC_parts:LCSC_C492610_Fuse_holder -> LCSC_parts:LCSC_C2935870_Fuse_holder
- F122: renamed from F64; footprint LCSC_parts:LCSC_C492610_Fuse_holder -> LCSC_parts:LCSC_C2935870_Fuse_holder
- F123: renamed from F65; footprint LCSC_parts:LCSC_C492610_Fuse_holder -> LCSC_parts:LCSC_C2935870_Fuse_holder
- F124: renamed from F66; footprint LCSC_parts:LCSC_C492610_Fuse_holder -> LCSC_parts:LCSC_C2935870_Fuse_holder
- F125: renamed from F67; footprint LCSC_parts:LCSC_C492610_Fuse_holder -> LCSC_parts:LCSC_C2935870_Fuse_holder
- F126: renamed from F68; footprint LCSC_parts:LCSC_C492610_Fuse_holder -> LCSC_parts:LCSC_C2935870_Fuse_holder
- F127: renamed from F69; footprint LCSC_parts:LCSC_C492610_Fuse_holder -> LCSC_parts:LCSC_C2935870_Fuse_holder
- F128: renamed from F70; footprint LCSC_parts:LCSC_C492610_Fuse_holder -> LCSC_parts:LCSC_C2935870_Fuse_holder
- F129: renamed from F71; footprint LCSC_parts:LCSC_C492610_Fuse_holder -> LCSC_parts:LCSC_C2935870_Fuse_holder
- F130: renamed from F72; footprint LCSC_parts:LCSC_C492610_Fuse_holder -> LCSC_parts:LCSC_C2935870_Fuse_holder
- F131: renamed from F73; footprint LCSC_parts:LCSC_C492610_Fuse_holder -> LCSC_parts:LCSC_C2935870_Fuse_holder
- F132: renamed from F74; footprint LCSC_parts:LCSC_C492610_Fuse_holder -> LCSC_parts:LCSC_C2935870_Fuse_holder
- F201: renamed from F12; footprint LCSC_parts:LCSC_C492610_Fuse_holder -> LCSC_parts:LCSC_C2935870_Fuse_holder
- F202: renamed from F13; footprint LCSC_parts:LCSC_C492610_Fuse_holder -> LCSC_parts:LCSC_C2935870_Fuse_holder
- F203: renamed from F14; footprint LCSC_parts:LCSC_C492610_Fuse_holder -> LCSC_parts:LCSC_C2935870_Fuse_holder
- F204: renamed from F15; footprint LCSC_parts:LCSC_C492610_Fuse_holder -> LCSC_parts:LCSC_C2935870_Fuse_holder
- F205: renamed from F16; footprint LCSC_parts:LCSC_C492610_Fuse_holder -> LCSC_parts:LCSC_C2935870_Fuse_holder
- F206: renamed from F17; footprint LCSC_parts:LCSC_C492610_Fuse_holder -> LCSC_parts:LCSC_C2935870_Fuse_holder
- F207: renamed from F18; footprint LCSC_parts:LCSC_C492610_Fuse_holder -> LCSC_parts:LCSC_C2935870_Fuse_holder
- F208: renamed from F19; footprint LCSC_parts:LCSC_C492610_Fuse_holder -> LCSC_parts:LCSC_C2935870_Fuse_holder
- F209: renamed from F20; footprint LCSC_parts:LCSC_C492610_Fuse_holder -> LCSC_parts:LCSC_C2935870_Fuse_holder
- F210: renamed from F21; footprint LCSC_parts:LCSC_C492610_Fuse_holder -> LCSC_parts:LCSC_C2935870_Fuse_holder
- F211: renamed from F22; footprint LCSC_parts:LCSC_C492610_Fuse_holder -> LCSC_parts:LCSC_C2935870_Fuse_holder
- F212: renamed from F44; footprint LCSC_parts:LCSC_C492610_Fuse_holder -> LCSC_parts:LCSC_C2935870_Fuse_holder
- F213: renamed from F45; footprint LCSC_parts:LCSC_C492610_Fuse_holder -> LCSC_parts:LCSC_C2935870_Fuse_holder
- F214: renamed from F46; footprint LCSC_parts:LCSC_C492610_Fuse_holder -> LCSC_parts:LCSC_C2935870_Fuse_holder
- F215: renamed from F47; footprint LCSC_parts:LCSC_C492610_Fuse_holder -> LCSC_parts:LCSC_C2935870_Fuse_holder
- F216: renamed from F48; footprint LCSC_parts:LCSC_C492610_Fuse_holder -> LCSC_parts:LCSC_C2935870_Fuse_holder
- F217: renamed from F49; footprint LCSC_parts:LCSC_C492610_Fuse_holder -> LCSC_parts:LCSC_C2935870_Fuse_holder
- F218: renamed from F50; footprint LCSC_parts:LCSC_C492610_Fuse_holder -> LCSC_parts:LCSC_C2935870_Fuse_holder
- F219: renamed from F51; footprint LCSC_parts:LCSC_C492610_Fuse_holder -> LCSC_parts:LCSC_C2935870_Fuse_holder
- F220: renamed from F52; footprint LCSC_parts:LCSC_C492610_Fuse_holder -> LCSC_parts:LCSC_C2935870_Fuse_holder
- F221: renamed from F53; footprint LCSC_parts:LCSC_C492610_Fuse_holder -> LCSC_parts:LCSC_C2935870_Fuse_holder
- F222: renamed from F75; footprint LCSC_parts:LCSC_C492610_Fuse_holder -> LCSC_parts:LCSC_C2935870_Fuse_holder
- F223: renamed from F76; footprint LCSC_parts:LCSC_C492610_Fuse_holder -> LCSC_parts:LCSC_C2935870_Fuse_holder
- F224: renamed from F77; footprint LCSC_parts:LCSC_C492610_Fuse_holder -> LCSC_parts:LCSC_C2935870_Fuse_holder
- F225: renamed from F78; footprint LCSC_parts:LCSC_C492610_Fuse_holder -> LCSC_parts:LCSC_C2935870_Fuse_holder
- F226: renamed from F79; footprint LCSC_parts:LCSC_C492610_Fuse_holder -> LCSC_parts:LCSC_C2935870_Fuse_holder
- F227: renamed from F80; footprint LCSC_parts:LCSC_C492610_Fuse_holder -> LCSC_parts:LCSC_C2935870_Fuse_holder
- F228: renamed from F81; footprint LCSC_parts:LCSC_C492610_Fuse_holder -> LCSC_parts:LCSC_C2935870_Fuse_holder
- F229: renamed from F82; footprint LCSC_parts:LCSC_C492610_Fuse_holder -> LCSC_parts:LCSC_C2935870_Fuse_holder
- F230: renamed from F83; footprint LCSC_parts:LCSC_C492610_Fuse_holder -> LCSC_parts:LCSC_C2935870_Fuse_holder
- F231: renamed from F84; footprint LCSC_parts:LCSC_C492610_Fuse_holder -> LCSC_parts:LCSC_C2935870_Fuse_holder
- F232: renamed from F85; footprint LCSC_parts:LCSC_C492610_Fuse_holder -> LCSC_parts:LCSC_C2935870_Fuse_holder
- F301: renamed from F23; footprint LCSC_parts:LCSC_C492610_Fuse_holder -> LCSC_parts:LCSC_C2935870_Fuse_holder
- F302: renamed from F24; footprint LCSC_parts:LCSC_C492610_Fuse_holder -> LCSC_parts:LCSC_C2935870_Fuse_holder
- F303: renamed from F25; footprint LCSC_parts:LCSC_C492610_Fuse_holder -> LCSC_parts:LCSC_C2935870_Fuse_holder
- F304: renamed from F26; footprint LCSC_parts:LCSC_C492610_Fuse_holder -> LCSC_parts:LCSC_C2935870_Fuse_holder
- F305: renamed from F27; footprint LCSC_parts:LCSC_C492610_Fuse_holder -> LCSC_parts:LCSC_C2935870_Fuse_holder
- F306: renamed from F28; footprint LCSC_parts:LCSC_C492610_Fuse_holder -> LCSC_parts:LCSC_C2935870_Fuse_holder
- F307: renamed from F29; footprint LCSC_parts:LCSC_C492610_Fuse_holder -> LCSC_parts:LCSC_C2935870_Fuse_holder
- F308: renamed from F30; footprint LCSC_parts:LCSC_C492610_Fuse_holder -> LCSC_parts:LCSC_C2935870_Fuse_holder
- F309: renamed from F31; footprint LCSC_parts:LCSC_C492610_Fuse_holder -> LCSC_parts:LCSC_C2935870_Fuse_holder
- F310: renamed from F32; footprint LCSC_parts:LCSC_C492610_Fuse_holder -> LCSC_parts:LCSC_C2935870_Fuse_holder
- F311: renamed from F33; footprint LCSC_parts:LCSC_C492610_Fuse_holder -> LCSC_parts:LCSC_C2935870_Fuse_holder
- F312: renamed from F54; footprint LCSC_parts:LCSC_C492610_Fuse_holder -> LCSC_parts:LCSC_C2935870_Fuse_holder
- F313: renamed from F55; footprint LCSC_parts:LCSC_C492610_Fuse_holder -> LCSC_parts:LCSC_C2935870_Fuse_holder
- F314: renamed from F56; footprint LCSC_parts:LCSC_C492610_Fuse_holder -> LCSC_parts:LCSC_C2935870_Fuse_holder
- F315: renamed from F57; footprint LCSC_parts:LCSC_C492610_Fuse_holder -> LCSC_parts:LCSC_C2935870_Fuse_holder
- F316: renamed from F58; footprint LCSC_parts:LCSC_C492610_Fuse_holder -> LCSC_parts:LCSC_C2935870_Fuse_holder
- F317: renamed from F59; footprint LCSC_parts:LCSC_C492610_Fuse_holder -> LCSC_parts:LCSC_C2935870_Fuse_holder
- F318: renamed from F60; footprint LCSC_parts:LCSC_C492610_Fuse_holder -> LCSC_parts:LCSC_C2935870_Fuse_holder
- F319: renamed from F61; footprint LCSC_parts:LCSC_C492610_Fuse_holder -> LCSC_parts:LCSC_C2935870_Fuse_holder
- F320: renamed from F62; footprint LCSC_parts:LCSC_C492610_Fuse_holder -> LCSC_parts:LCSC_C2935870_Fuse_holder
- F321: renamed from F63; footprint LCSC_parts:LCSC_C492610_Fuse_holder -> LCSC_parts:LCSC_C2935870_Fuse_holder
- F322: renamed from F86; footprint LCSC_parts:LCSC_C492610_Fuse_holder -> LCSC_parts:LCSC_C2935870_Fuse_holder
- F323: renamed from F87; footprint LCSC_parts:LCSC_C492610_Fuse_holder -> LCSC_parts:LCSC_C2935870_Fuse_holder
- F324: renamed from F88; footprint LCSC_parts:LCSC_C492610_Fuse_holder -> LCSC_parts:LCSC_C2935870_Fuse_holder
- F325: renamed from F89; footprint LCSC_parts:LCSC_C492610_Fuse_holder -> LCSC_parts:LCSC_C2935870_Fuse_holder
- F326: renamed from F90; footprint LCSC_parts:LCSC_C492610_Fuse_holder -> LCSC_parts:LCSC_C2935870_Fuse_holder
- F327: renamed from F91; footprint LCSC_parts:LCSC_C492610_Fuse_holder -> LCSC_parts:LCSC_C2935870_Fuse_holder
- F328: renamed from F92; footprint LCSC_parts:LCSC_C492610_Fuse_holder -> LCSC_parts:LCSC_C2935870_Fuse_holder
- F329: renamed from F93; footprint LCSC_parts:LCSC_C492610_Fuse_holder -> LCSC_parts:LCSC_C2935870_Fuse_holder
- F330: renamed from F94; footprint LCSC_parts:LCSC_C492610_Fuse_holder -> LCSC_parts:LCSC_C2935870_Fuse_holder
- F331: renamed from F95; footprint LCSC_parts:LCSC_C492610_Fuse_holder -> LCSC_parts:LCSC_C2935870_Fuse_holder
- F332: renamed from F96; footprint LCSC_parts:LCSC_C492610_Fuse_holder -> LCSC_parts:LCSC_C2935870_Fuse_holder
- F401: renamed from F97; footprint LCSC_parts:LCSC_C492610_Fuse_holder -> LCSC_parts:LCSC_C2935870_Fuse_holder
- F402: renamed from F98; footprint LCSC_parts:LCSC_C492610_Fuse_holder -> LCSC_parts:LCSC_C2935870_Fuse_holder
- F403: renamed from F99; footprint LCSC_parts:LCSC_C492610_Fuse_holder -> LCSC_parts:LCSC_C2935870_Fuse_holder
- F404: renamed from F100; footprint LCSC_parts:LCSC_C492610_Fuse_holder -> LCSC_parts:LCSC_C2935870_Fuse_holder
- F405: renamed from F101; footprint LCSC_parts:LCSC_C492610_Fuse_holder -> LCSC_parts:LCSC_C2935870_Fuse_holder
- F406: renamed from F102; footprint LCSC_parts:LCSC_C492610_Fuse_holder -> LCSC_parts:LCSC_C2935870_Fuse_holder
- F407: renamed from F103; footprint LCSC_parts:LCSC_C492610_Fuse_holder -> LCSC_parts:LCSC_C2935870_Fuse_holder
- F408: renamed from F104; footprint LCSC_parts:LCSC_C492610_Fuse_holder -> LCSC_parts:LCSC_C2935870_Fuse_holder
- F409: renamed from F105; footprint LCSC_parts:LCSC_C492610_Fuse_holder -> LCSC_parts:LCSC_C2935870_Fuse_holder
- F410: renamed from F106; footprint LCSC_parts:LCSC_C492610_Fuse_holder -> LCSC_parts:LCSC_C2935870_Fuse_holder
- F411: renamed from F107; footprint LCSC_parts:LCSC_C492610_Fuse_holder -> LCSC_parts:LCSC_C2935870_Fuse_holder
- F412: renamed from F130; footprint LCSC_parts:LCSC_C492610_Fuse_holder -> LCSC_parts:LCSC_C2935870_Fuse_holder
- F413: renamed from F131; footprint LCSC_parts:LCSC_C492610_Fuse_holder -> LCSC_parts:LCSC_C2935870_Fuse_holder
- F414: renamed from F132; footprint LCSC_parts:LCSC_C492610_Fuse_holder -> LCSC_parts:LCSC_C2935870_Fuse_holder
- F415: renamed from F133; footprint LCSC_parts:LCSC_C492610_Fuse_holder -> LCSC_parts:LCSC_C2935870_Fuse_holder
- F416: renamed from F134; footprint LCSC_parts:LCSC_C492610_Fuse_holder -> LCSC_parts:LCSC_C2935870_Fuse_holder
- F417: renamed from F135; footprint LCSC_parts:LCSC_C492610_Fuse_holder -> LCSC_parts:LCSC_C2935870_Fuse_holder
- F418: renamed from F136; footprint LCSC_parts:LCSC_C492610_Fuse_holder -> LCSC_parts:LCSC_C2935870_Fuse_holder
- F419: renamed from F137; footprint LCSC_parts:LCSC_C492610_Fuse_holder -> LCSC_parts:LCSC_C2935870_Fuse_holder
- F420: renamed from F138; footprint LCSC_parts:LCSC_C492610_Fuse_holder -> LCSC_parts:LCSC_C2935870_Fuse_holder
- F421: renamed from F139; footprint LCSC_parts:LCSC_C492610_Fuse_holder -> LCSC_parts:LCSC_C2935870_Fuse_holder
- F422: renamed from F160; footprint LCSC_parts:LCSC_C492610_Fuse_holder -> LCSC_parts:LCSC_C2935870_Fuse_holder
- F423: renamed from F161; footprint LCSC_parts:LCSC_C492610_Fuse_holder -> LCSC_parts:LCSC_C2935870_Fuse_holder
- F424: renamed from F162; footprint LCSC_parts:LCSC_C492610_Fuse_holder -> LCSC_parts:LCSC_C2935870_Fuse_holder
- F425: renamed from F163; footprint LCSC_parts:LCSC_C492610_Fuse_holder -> LCSC_parts:LCSC_C2935870_Fuse_holder
- F426: renamed from F164; footprint LCSC_parts:LCSC_C492610_Fuse_holder -> LCSC_parts:LCSC_C2935870_Fuse_holder
- F427: renamed from F165; footprint LCSC_parts:LCSC_C492610_Fuse_holder -> LCSC_parts:LCSC_C2935870_Fuse_holder
- F428: renamed from F166; footprint LCSC_parts:LCSC_C492610_Fuse_holder -> LCSC_parts:LCSC_C2935870_Fuse_holder
- F429: renamed from F167; footprint LCSC_parts:LCSC_C492610_Fuse_holder -> LCSC_parts:LCSC_C2935870_Fuse_holder
- F430: renamed from F168; footprint LCSC_parts:LCSC_C492610_Fuse_holder -> LCSC_parts:LCSC_C2935870_Fuse_holder
- F431: renamed from F169; footprint LCSC_parts:LCSC_C492610_Fuse_holder -> LCSC_parts:LCSC_C2935870_Fuse_holder
- F432: renamed from F170; footprint LCSC_parts:LCSC_C492610_Fuse_holder -> LCSC_parts:LCSC_C2935870_Fuse_holder
- F501: renamed from F108; footprint LCSC_parts:LCSC_C492610_Fuse_holder -> LCSC_parts:LCSC_C2935870_Fuse_holder
- F502: renamed from F109; footprint LCSC_parts:LCSC_C492610_Fuse_holder -> LCSC_parts:LCSC_C2935870_Fuse_holder
- F503: renamed from F110; footprint LCSC_parts:LCSC_C492610_Fuse_holder -> LCSC_parts:LCSC_C2935870_Fuse_holder
- F504: renamed from F111; footprint LCSC_parts:LCSC_C492610_Fuse_holder -> LCSC_parts:LCSC_C2935870_Fuse_holder
- F505: renamed from F112; footprint LCSC_parts:LCSC_C492610_Fuse_holder -> LCSC_parts:LCSC_C2935870_Fuse_holder
- F506: renamed from F113; footprint LCSC_parts:LCSC_C492610_Fuse_holder -> LCSC_parts:LCSC_C2935870_Fuse_holder
- F507: renamed from F114; footprint LCSC_parts:LCSC_C492610_Fuse_holder -> LCSC_parts:LCSC_C2935870_Fuse_holder
- F508: renamed from F115; footprint LCSC_parts:LCSC_C492610_Fuse_holder -> LCSC_parts:LCSC_C2935870_Fuse_holder
- F509: renamed from F116; footprint LCSC_parts:LCSC_C492610_Fuse_holder -> LCSC_parts:LCSC_C2935870_Fuse_holder
- F510: renamed from F117; footprint LCSC_parts:LCSC_C492610_Fuse_holder -> LCSC_parts:LCSC_C2935870_Fuse_holder
- F511: renamed from F118; footprint LCSC_parts:LCSC_C492610_Fuse_holder -> LCSC_parts:LCSC_C2935870_Fuse_holder
- F512: renamed from F140; footprint LCSC_parts:LCSC_C492610_Fuse_holder -> LCSC_parts:LCSC_C2935870_Fuse_holder
- F513: renamed from F141; footprint LCSC_parts:LCSC_C492610_Fuse_holder -> LCSC_parts:LCSC_C2935870_Fuse_holder
- F514: renamed from F142; footprint LCSC_parts:LCSC_C492610_Fuse_holder -> LCSC_parts:LCSC_C2935870_Fuse_holder
- F515: renamed from F143; footprint LCSC_parts:LCSC_C492610_Fuse_holder -> LCSC_parts:LCSC_C2935870_Fuse_holder
- F516: renamed from F144; footprint LCSC_parts:LCSC_C492610_Fuse_holder -> LCSC_parts:LCSC_C2935870_Fuse_holder
- F517: renamed from F145; footprint LCSC_parts:LCSC_C492610_Fuse_holder -> LCSC_parts:LCSC_C2935870_Fuse_holder
- F518: renamed from F146; footprint LCSC_parts:LCSC_C492610_Fuse_holder -> LCSC_parts:LCSC_C2935870_Fuse_holder
- F519: renamed from F147; footprint LCSC_parts:LCSC_C492610_Fuse_holder -> LCSC_parts:LCSC_C2935870_Fuse_holder
- F520: renamed from F148; footprint LCSC_parts:LCSC_C492610_Fuse_holder -> LCSC_parts:LCSC_C2935870_Fuse_holder
- F521: renamed from F149; footprint LCSC_parts:LCSC_C492610_Fuse_holder -> LCSC_parts:LCSC_C2935870_Fuse_holder
- F522: renamed from F171; footprint LCSC_parts:LCSC_C492610_Fuse_holder -> LCSC_parts:LCSC_C2935870_Fuse_holder
- F523: renamed from F172; footprint LCSC_parts:LCSC_C492610_Fuse_holder -> LCSC_parts:LCSC_C2935870_Fuse_holder
- F524: renamed from F173; footprint LCSC_parts:LCSC_C492610_Fuse_holder -> LCSC_parts:LCSC_C2935870_Fuse_holder
- F525: renamed from F174; footprint LCSC_parts:LCSC_C492610_Fuse_holder -> LCSC_parts:LCSC_C2935870_Fuse_holder
- F526: renamed from F175; footprint LCSC_parts:LCSC_C492610_Fuse_holder -> LCSC_parts:LCSC_C2935870_Fuse_holder
- F527: renamed from F176; footprint LCSC_parts:LCSC_C492610_Fuse_holder -> LCSC_parts:LCSC_C2935870_Fuse_holder
- F528: renamed from F177; footprint LCSC_parts:LCSC_C492610_Fuse_holder -> LCSC_parts:LCSC_C2935870_Fuse_holder
- F529: renamed from F178; footprint LCSC_parts:LCSC_C492610_Fuse_holder -> LCSC_parts:LCSC_C2935870_Fuse_holder
- F530: renamed from F179; footprint LCSC_parts:LCSC_C492610_Fuse_holder -> LCSC_parts:LCSC_C2935870_Fuse_holder
- F531: renamed from F180; footprint LCSC_parts:LCSC_C492610_Fuse_holder -> LCSC_parts:LCSC_C2935870_Fuse_holder
- F532: renamed from F181; footprint LCSC_parts:LCSC_C492610_Fuse_holder -> LCSC_parts:LCSC_C2935870_Fuse_holder
- F601: renamed from F119; footprint LCSC_parts:LCSC_C492610_Fuse_holder -> LCSC_parts:LCSC_C2935870_Fuse_holder
- F602: renamed from F120; footprint LCSC_parts:LCSC_C492610_Fuse_holder -> LCSC_parts:LCSC_C2935870_Fuse_holder
- F603: renamed from F121; footprint LCSC_parts:LCSC_C492610_Fuse_holder -> LCSC_parts:LCSC_C2935870_Fuse_holder
- F604: renamed from F122; footprint LCSC_parts:LCSC_C492610_Fuse_holder -> LCSC_parts:LCSC_C2935870_Fuse_holder
- F605: renamed from F123; footprint LCSC_parts:LCSC_C492610_Fuse_holder -> LCSC_parts:LCSC_C2935870_Fuse_holder
- F606: renamed from F124; footprint LCSC_parts:LCSC_C492610_Fuse_holder -> LCSC_parts:LCSC_C2935870_Fuse_holder
- F607: renamed from F125; footprint LCSC_parts:LCSC_C492610_Fuse_holder -> LCSC_parts:LCSC_C2935870_Fuse_holder
- F608: renamed from F126; footprint LCSC_parts:LCSC_C492610_Fuse_holder -> LCSC_parts:LCSC_C2935870_Fuse_holder
- F609: renamed from F127; footprint LCSC_parts:LCSC_C492610_Fuse_holder -> LCSC_parts:LCSC_C2935870_Fuse_holder
- F610: renamed from F128; footprint LCSC_parts:LCSC_C492610_Fuse_holder -> LCSC_parts:LCSC_C2935870_Fuse_holder
- F611: renamed from F129; footprint LCSC_parts:LCSC_C492610_Fuse_holder -> LCSC_parts:LCSC_C2935870_Fuse_holder
- F612: renamed from F150; footprint LCSC_parts:LCSC_C492610_Fuse_holder -> LCSC_parts:LCSC_C2935870_Fuse_holder
- F613: renamed from F151; footprint LCSC_parts:LCSC_C492610_Fuse_holder -> LCSC_parts:LCSC_C2935870_Fuse_holder
- F614: renamed from F152; footprint LCSC_parts:LCSC_C492610_Fuse_holder -> LCSC_parts:LCSC_C2935870_Fuse_holder
- F615: renamed from F153; footprint LCSC_parts:LCSC_C492610_Fuse_holder -> LCSC_parts:LCSC_C2935870_Fuse_holder
- F616: renamed from F154; footprint LCSC_parts:LCSC_C492610_Fuse_holder -> LCSC_parts:LCSC_C2935870_Fuse_holder
- F617: renamed from F155; footprint LCSC_parts:LCSC_C492610_Fuse_holder -> LCSC_parts:LCSC_C2935870_Fuse_holder
- F618: renamed from F156; footprint LCSC_parts:LCSC_C492610_Fuse_holder -> LCSC_parts:LCSC_C2935870_Fuse_holder
- F619: renamed from F157; footprint LCSC_parts:LCSC_C492610_Fuse_holder -> LCSC_parts:LCSC_C2935870_Fuse_holder
- F620: renamed from F158; footprint LCSC_parts:LCSC_C492610_Fuse_holder -> LCSC_parts:LCSC_C2935870_Fuse_holder
- F621: renamed from F159; footprint LCSC_parts:LCSC_C492610_Fuse_holder -> LCSC_parts:LCSC_C2935870_Fuse_holder
- F622: renamed from F182; footprint LCSC_parts:LCSC_C492610_Fuse_holder -> LCSC_parts:LCSC_C2935870_Fuse_holder
- F623: renamed from F183; footprint LCSC_parts:LCSC_C492610_Fuse_holder -> LCSC_parts:LCSC_C2935870_Fuse_holder
- F624: renamed from F184; footprint LCSC_parts:LCSC_C492610_Fuse_holder -> LCSC_parts:LCSC_C2935870_Fuse_holder
- F625: renamed from F185; footprint LCSC_parts:LCSC_C492610_Fuse_holder -> LCSC_parts:LCSC_C2935870_Fuse_holder
- F626: renamed from F186; footprint LCSC_parts:LCSC_C492610_Fuse_holder -> LCSC_parts:LCSC_C2935870_Fuse_holder
- F627: renamed from F187; footprint LCSC_parts:LCSC_C492610_Fuse_holder -> LCSC_parts:LCSC_C2935870_Fuse_holder
- F628: renamed from F188; footprint LCSC_parts:LCSC_C492610_Fuse_holder -> LCSC_parts:LCSC_C2935870_Fuse_holder
- F629: renamed from F189; footprint LCSC_parts:LCSC_C492610_Fuse_holder -> LCSC_parts:LCSC_C2935870_Fuse_holder
- F630: renamed from F190; footprint LCSC_parts:LCSC_C492610_Fuse_holder -> LCSC_parts:LCSC_C2935870_Fuse_holder
- F631: renamed from F191; footprint LCSC_parts:LCSC_C492610_Fuse_holder -> LCSC_parts:LCSC_C2935870_Fuse_holder
- F632: renamed from F192; footprint LCSC_parts:LCSC_C492610_Fuse_holder -> LCSC_parts:LCSC_C2935870_Fuse_holder
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- renumbered TP1 to TP101, TP2 to TP102, TP3 to TP103, TP4 to TP104, TP5 to TP105, TP6 to TP106, TP7 to TP107, TP8 to TP108, TP9 to TP109, TP10 to TP110, TP11 to TP111, TP34 to TP112, TP35 to TP113, TP36 to TP114, TP37 to TP115, TP38 to TP116, TP39 to TP117, TP40 to TP118, TP42 to TP119, TP43 to TP120, TP44 to TP121, TP67 to TP122, TP68 to TP123, TP69 to TP124, TP70 to TP125, TP71 to TP126, TP72 to TP127, TP73 to TP128, TP74 to TP129, TP75 to TP130, TP76 to TP131, TP77 to TP132, TP12 to TP201, TP13 to TP202, TP14 to TP203, TP15 to TP204, TP16 to TP205, TP17 to TP206, TP18 to TP207, TP19 to TP208, TP20 to TP209, TP21 to TP210, TP22 to TP211, TP45 to TP212, TP46 to TP213, TP47 to TP214, TP48 to TP215, TP49 to TP216, TP50 to TP217, TP51 to TP218, TP52 to TP219, TP53 to TP220, TP54 to TP221, TP78 to TP222, TP79 to TP223, TP80 to TP224, TP81 to TP225, TP82 to TP226, TP83 to TP227, TP84 to TP228, TP85 to TP229, TP86 to TP230, TP87 to TP231, TP88 to TP232, TP23 to TP301, TP24 to TP302, TP25 to TP303, TP26 to TP304, TP27 to TP305, TP28 to TP306, TP29 to TP307, TP30 to TP308, TP31 to TP309, TP32 to TP310, TP33 to TP311, TP56 to TP312, TP57 to TP313, TP58 to TP314, TP59 to TP315, TP60 to TP316, TP61 to TP317, TP62 to TP318, TP63 to TP319, TP64 to TP320, TP65 to TP321, TP89 to TP322, TP90 to TP323, TP91 to TP324, TP92 to TP325, TP93 to TP326, TP94 to TP327, TP95 to TP328, TP96 to TP329, TP97 to TP330, TP98 to TP331, TP99 to TP332, TP100 to TP401, TP101 to TP402, TP102 to TP403, TP103 to TP404, TP104 to TP405, TP105 to TP406, TP106 to TP407, TP107 to TP408, TP108 to TP409, TP109 to TP410, TP110 to TP411, TP133 to TP412, TP134 to TP413, TP135 to TP414, TP136 to TP415, TP137 to TP416, TP138 to TP417, TP139 to TP418, TP140 to TP419, TP141 to TP420, TP142 to TP421, TP166 to TP422, TP167 to TP423, TP168 to TP424, TP169 to TP425, TP170 to TP426, TP171 to TP427, TP172 to TP428, TP173 to TP429, TP174 to TP430, TP175 to TP431, TP176 to TP432, TP111 to TP501, TP112 to TP502, TP113 to TP503, TP114 to TP504, TP115 to TP505, TP116 to TP506, TP117 to TP507, TP118 to TP508, TP119 to TP509, TP120 to TP510, TP121 to TP511, TP144 to TP512, TP145 to TP513, TP146 to TP514, TP147 to TP515, TP148 to TP516, TP149 to TP517, TP150 to TP518, TP151 to TP519, TP152 to TP520, TP153 to TP521, TP177 to TP522, TP178 to TP523, TP179 to TP524, TP180 to TP525, TP181 to TP526, TP182 to TP527, TP183 to TP528, TP184 to TP529, TP185 to TP530, TP186 to TP531, TP187 to TP532, TP122 to TP601, TP123 to TP602, TP124 to TP603, TP125 to TP604, TP126 to TP605, TP127 to TP606, TP128 to TP607, TP129 to TP608, TP130 to TP609, TP131 to TP610, TP132 to TP611, TP155 to TP612, TP156 to TP613, TP157 to TP614, TP158 to TP615, TP159 to TP616, TP160 to TP617, TP161 to TP618, TP162 to TP619, TP163 to TP620, TP164 to TP621, TP188 to TP622, TP189 to TP623, TP190 to TP624, TP191 to TP625, TP192 to TP626, TP41 to TP627, TP55 to TP628, TP154 to TP629, TP143 to TP630, TP165 to TP631, TP66 to TP632
Connections:
- F112 pad 2: Net-(F130-Pad1) -> Net-(F112-Pad2)
- F113 pad 2: Net-(F131-Pad1) -> Net-(F113-Pad2)
- F114 pad 2: Net-(F132-Pad1) -> Net-(F114-Pad2)
- F115 pad 2: Net-(F133-Pad1) -> Net-(F115-Pad2)
- F116 pad 2: Net-(F134-Pad1) -> Net-(F116-Pad2)
- F117 pad 2: Net-(F135-Pad1) -> Net-(F117-Pad2)
- F118 pad 2: Net-(F136-Pad1) -> Net-(F118-Pad2)
- F119 pad 1: Net-(F41-Pad1) -> Net-(F119-Pad1)
- F119 pad 2: Net-(F137-Pad1) -> Net-(F119-Pad2)
- F120 pad 1: Net-(F42-Pad1) -> Net-(F120-Pad1)
- F120 pad 2: Net-(F138-Pad1) -> Net-(F120-Pad2)
- F121 pad 1: Net-(F43-Pad1) -> Net-(F121-Pad1)
- F121 pad 2: Net-(F139-Pad1) -> Net-(F121-Pad2)
- F122 pad 1: Net-(F64-Pad1) -> Net-(F122-Pad1)
- F122 pad 2: Net-(F160-Pad1) -> Net-(F122-Pad2)
- F123 pad 1: Net-(F65-Pad1) -> Net-(F123-Pad1)
- F123 pad 2: Net-(F161-Pad1) -> Net-(F123-Pad2)
- F124 pad 1: Net-(F66-Pad1) -> Net-(F124-Pad1)
- F124 pad 2: Net-(F162-Pad1) -> Net-(F124-Pad2)
- F125 pad 1: Net-(F67-Pad1) -> Net-(F125-Pad1)
- F125 pad 2: Net-(F163-Pad1) -> Net-(F125-Pad2)
- F126 pad 1: Net-(F68-Pad1) -> Net-(F126-Pad1)
- F126 pad 2: Net-(F164-Pad1) -> Net-(F126-Pad2)
- F127 pad 1: Net-(F69-Pad1) -> Net-(F127-Pad1)
- F127 pad 2: Net-(F165-Pad1) -> Net-(F127-Pad2)
- F128 pad 1: Net-(F70-Pad1) -> Net-(F128-Pad1)
- F128 pad 2: Net-(F166-Pad1) -> Net-(F128-Pad2)
- F129 pad 1: Net-(F71-Pad1) -> Net-(F129-Pad1)
- F129 pad 2: Net-(F167-Pad1) -> Net-(F129-Pad2)
- F130 pad 1: Net-(F72-Pad1) -> Net-(F130-Pad1)
- F130 pad 2: Net-(F168-Pad1) -> Net-(F130-Pad2)
- F131 pad 1: Net-(F73-Pad1) -> Net-(F131-Pad1)
- F131 pad 2: Net-(F169-Pad1) -> Net-(F131-Pad2)
- F132 pad 1: Net-(F74-Pad1) -> Net-(F132-Pad1)
- F132 pad 2: Net-(F170-Pad1) -> Net-(F132-Pad2)
- F201 pad 2: Net-(F108-Pad1) (its old number) -> Net-(F201-Pad2)
- F202 pad 2: Net-(F109-Pad1) (its old number) -> Net-(F202-Pad2)
- F203 pad 2: Net-(F110-Pad1) (its old number) -> Net-(F203-Pad2)
- F204 pad 2: Net-(F111-Pad1) (its old number) -> Net-(F204-Pad2)
- F205 pad 2: Net-(F112-Pad1) (its old number) -> Net-(F205-Pad2)
- F206 pad 2: Net-(F113-Pad1) (its old number) -> Net-(F206-Pad2)
- F207 pad 2: Net-(F114-Pad1) (its old number) -> Net-(F207-Pad2)
- F208 pad 2: Net-(F115-Pad1) (its old number) -> Net-(F208-Pad2)
- F209 pad 2: Net-(F116-Pad1) (its old number) -> Net-(F209-Pad2)
- F210 pad 2: Net-(F117-Pad1) (its old number) -> Net-(F210-Pad2)
- F211 pad 2: Net-(F118-Pad1) (its old number) -> Net-(F211-Pad2)
- F212 pad 1: Net-(F44-Pad1) -> Net-(F212-Pad1)
- F213 pad 1: Net-(F45-Pad1) -> Net-(F213-Pad1)
- F214 pad 1: Net-(F46-Pad1) -> Net-(F214-Pad1)
- F215 pad 1: Net-(F47-Pad1) -> Net-(F215-Pad1)
- F216 pad 1: Net-(F48-Pad1) -> Net-(F216-Pad1)
- F217 pad 1: Net-(F49-Pad1) -> Net-(F217-Pad1)
- F218 pad 1: Net-(F50-Pad1) -> Net-(F218-Pad1)
- F219 pad 1: Net-(F51-Pad1) -> Net-(F219-Pad1)
- F220 pad 1: Net-(F52-Pad1) -> Net-(F220-Pad1)
- F221 pad 1: Net-(F53-Pad1) -> Net-(F221-Pad1)
- F222 pad 1: Net-(F75-Pad1) -> Net-(F222-Pad1)
- F222 pad 2: Net-(F171-Pad1) -> Net-(F222-Pad2)
- F223 pad 1: Net-(F76-Pad1) -> Net-(F223-Pad1)
- F223 pad 2: Net-(F172-Pad1) -> Net-(F223-Pad2)
- F224 pad 1: Net-(F77-Pad1) -> Net-(F224-Pad1)
- F224 pad 2: Net-(F173-Pad1) -> Net-(F224-Pad2)
- F225 pad 1: Net-(F78-Pad1) -> Net-(F225-Pad1)
- F225 pad 2: Net-(F174-Pad1) -> Net-(F225-Pad2)
- F226 pad 1: Net-(F79-Pad1) -> Net-(F226-Pad1)
- F226 pad 2: Net-(F175-Pad1) -> Net-(F226-Pad2)
- F227 pad 1: Net-(F80-Pad1) -> Net-(F227-Pad1)
- F227 pad 2: Net-(F176-Pad1) -> Net-(F227-Pad2)
- F228 pad 1: Net-(F81-Pad1) -> Net-(F228-Pad1)
- F228 pad 2: Net-(F177-Pad1) -> Net-(F228-Pad2)
- F229 pad 1: Net-(F82-Pad1) -> Net-(F229-Pad1)
- F229 pad 2: Net-(F178-Pad1) -> Net-(F229-Pad2)
- F230 pad 1: Net-(F83-Pad1) -> Net-(F230-Pad1)
- F230 pad 2: Net-(F179-Pad1) -> Net-(F230-Pad2)
- F231 pad 1: Net-(F84-Pad1) -> Net-(F231-Pad1)
- F231 pad 2: Net-(F180-Pad1) -> Net-(F231-Pad2)
- F232 pad 1: Net-(F85-Pad1) -> Net-(F232-Pad1)
- F232 pad 2: Net-(F181-Pad1) -> Net-(F232-Pad2)
- F301 pad 2: Net-(F119-Pad1) -> Net-(F301-Pad2)
- F302 pad 2: Net-(F120-Pad1) -> Net-(F302-Pad2)
- F303 pad 2: Net-(F121-Pad1) -> Net-(F303-Pad2)
- F304 pad 2: Net-(F122-Pad1) -> Net-(F304-Pad2)
- F305 pad 2: Net-(F123-Pad1) -> Net-(F305-Pad2)
- F306 pad 2: Net-(F124-Pad1) -> Net-(F306-Pad2)
- F307 pad 2: Net-(F125-Pad1) -> Net-(F307-Pad2)
- F308 pad 2: Net-(F126-Pad1) -> Net-(F308-Pad2)
- F309 pad 2: Net-(F127-Pad1) -> Net-(F309-Pad2)
- F310 pad 2: Net-(F128-Pad1) -> Net-(F310-Pad2)
- F311 pad 2: Net-(F129-Pad1) -> Net-(F311-Pad2)
- F312 pad 1: Net-(F54-Pad1) -> Net-(F312-Pad1)
- F312 pad 2: Net-(F150-Pad1) -> Net-(F312-Pad2)
- F313 pad 1: Net-(F55-Pad1) -> Net-(F313-Pad1)
- F313 pad 2: Net-(F151-Pad1) -> Net-(F313-Pad2)
- F314 pad 1: Net-(F56-Pad1) -> Net-(F314-Pad1)
- F314 pad 2: Net-(F152-Pad1) -> Net-(F314-Pad2)
- F315 pad 1: Net-(F57-Pad1) -> Net-(F315-Pad1)
- F315 pad 2: Net-(F153-Pad1) -> Net-(F315-Pad2)
- F316 pad 1: Net-(F58-Pad1) -> Net-(F316-Pad1)
- F316 pad 2: Net-(F154-Pad1) -> Net-(F316-Pad2)
- F317 pad 1: Net-(F59-Pad1) -> Net-(F317-Pad1)
- F317 pad 2: Net-(F155-Pad1) -> Net-(F317-Pad2)
- F318 pad 1: Net-(F60-Pad1) -> Net-(F318-Pad1)
- F318 pad 2: Net-(F156-Pad1) -> Net-(F318-Pad2)
- F319 pad 1: Net-(F61-Pad1) -> Net-(F319-Pad1)
- F319 pad 2: Net-(F157-Pad1) -> Net-(F319-Pad2)
- F320 pad 1: Net-(F62-Pad1) -> Net-(F320-Pad1)
- F320 pad 2: Net-(F158-Pad1) -> Net-(F320-Pad2)
- F321 pad 1: Net-(F63-Pad1) -> Net-(F321-Pad1)
- F321 pad 2: Net-(F159-Pad1) -> Net-(F321-Pad2)
- F322 pad 1: Net-(F86-Pad1) -> Net-(F322-Pad1)
- F323 pad 1: Net-(F87-Pad1) -> Net-(F323-Pad1)
- F324 pad 1: Net-(F88-Pad1) -> Net-(F324-Pad1)
- F325 pad 1: Net-(F89-Pad1) -> Net-(F325-Pad1)
- F326 pad 1: Net-(F90-Pad1) -> Net-(F326-Pad1)
- F327 pad 1: Net-(F91-Pad1) -> Net-(F327-Pad1)
- F328 pad 1: Net-(F92-Pad1) -> Net-(F328-Pad1)
- F329 pad 1: Net-(F93-Pad1) -> Net-(F329-Pad1)
- F330 pad 1: Net-(F94-Pad1) -> Net-(F330-Pad1)
- F331 pad 1: Net-(F95-Pad1) -> Net-(F331-Pad1)
- F332 pad 1: Net-(F96-Pad1) -> Net-(F332-Pad1)
- F401 pad 2: Net-(F97-Pad2) -> Net-(F401-Pad2)
- F402 pad 2: Net-(F98-Pad2) -> Net-(F402-Pad2)
- F403 pad 2: Net-(F99-Pad2) -> Net-(F403-Pad2)
- F404 pad 2: Net-(F100-Pad2) -> Net-(F404-Pad2)
- F405 pad 2: Net-(F101-Pad2) (its old number) -> Net-(F405-Pad2)
- F406 pad 2: Net-(F102-Pad2) (its old number) -> Net-(F406-Pad2)
- F407 pad 2: Net-(F103-Pad2) (its old number) -> Net-(F407-Pad2)
- F408 pad 2: Net-(F104-Pad2) (its old number) -> Net-(F408-Pad2)
- F409 pad 2: Net-(F105-Pad2) (its old number) -> Net-(F409-Pad2)
- F410 pad 2: Net-(F106-Pad2) (its old number) -> Net-(F410-Pad2)
- F411 pad 2: Net-(F107-Pad2) (its old number) -> Net-(F411-Pad2)
- F412 pad 1: Net-(F130-Pad1) -> Net-(F112-Pad2)
- F412 pad 2: Net-(F130-Pad2) -> Net-(F412-Pad2)
- F413 pad 1: Net-(F131-Pad1) -> Net-(F113-Pad2)
- F413 pad 2: Net-(F131-Pad2) -> Net-(F413-Pad2)
- F414 pad 1: Net-(F132-Pad1) -> Net-(F114-Pad2)
- F414 pad 2: Net-(F132-Pad2) -> Net-(F414-Pad2)
- F415 pad 1: Net-(F133-Pad1) -> Net-(F115-Pad2)
- F415 pad 2: Net-(F133-Pad2) -> Net-(F415-Pad2)
- F416 pad 1: Net-(F134-Pad1) -> Net-(F116-Pad2)
- F416 pad 2: Net-(F134-Pad2) -> Net-(F416-Pad2)
- F417 pad 1: Net-(F135-Pad1) -> Net-(F117-Pad2)
- F417 pad 2: Net-(F135-Pad2) -> Net-(F417-Pad2)
- F418 pad 1: Net-(F136-Pad1) -> Net-(F118-Pad2)
- F418 pad 2: Net-(F136-Pad2) -> Net-(F418-Pad2)
- F419 pad 1: Net-(F137-Pad1) -> Net-(F119-Pad2)
- F419 pad 2: Net-(F137-Pad2) -> Net-(F419-Pad2)
- F420 pad 1: Net-(F138-Pad1) -> Net-(F120-Pad2)
- F420 pad 2: Net-(F138-Pad2) -> Net-(F420-Pad2)
- F421 pad 1: Net-(F139-Pad1) -> Net-(F121-Pad2)
- F421 pad 2: Net-(F139-Pad2) -> Net-(F421-Pad2)
- F422 pad 1: Net-(F160-Pad1) -> Net-(F122-Pad2)
- F422 pad 2: Net-(F160-Pad2) -> Net-(F422-Pad2)
- F423 pad 1: Net-(F161-Pad1) -> Net-(F123-Pad2)
- F423 pad 2: Net-(F161-Pad2) -> Net-(F423-Pad2)
- F424 pad 1: Net-(F162-Pad1) -> Net-(F124-Pad2)
- F424 pad 2: Net-(F162-Pad2) -> Net-(F424-Pad2)
- F425 pad 1: Net-(F163-Pad1) -> Net-(F125-Pad2)
- F425 pad 2: Net-(F163-Pad2) -> Net-(F425-Pad2)
- F426 pad 1: Net-(F164-Pad1) -> Net-(F126-Pad2)
- F426 pad 2: Net-(F164-Pad2) -> Net-(F426-Pad2)
- F427 pad 1: Net-(F165-Pad1) -> Net-(F127-Pad2)
- F427 pad 2: Net-(F165-Pad2) -> Net-(F427-Pad2)
- F428 pad 1: Net-(F166-Pad1) -> Net-(F128-Pad2)
- F428 pad 2: Net-(F166-Pad2) -> Net-(F428-Pad2)
- F429 pad 1: Net-(F167-Pad1) -> Net-(F129-Pad2)
- F429 pad 2: Net-(F167-Pad2) -> Net-(F429-Pad2)
- F430 pad 1: Net-(F168-Pad1) -> Net-(F130-Pad2)
- F430 pad 2: Net-(F168-Pad2) -> Net-(F430-Pad2)
- F431 pad 1: Net-(F169-Pad1) -> Net-(F131-Pad2)
- F431 pad 2: Net-(F169-Pad2) -> Net-(F431-Pad2)
- F432 pad 1: Net-(F170-Pad1) -> Net-(F132-Pad2)
- F432 pad 2: Net-(F170-Pad2) -> Net-(F432-Pad2)
- F501 pad 1: Net-(F108-Pad1) (its old number) -> Net-(F201-Pad2)
- F501 pad 2: Net-(F108-Pad2) (its old number) -> Net-(F501-Pad2)
- F502 pad 1: Net-(F109-Pad1) (its old number) -> Net-(F202-Pad2)
- F502 pad 2: Net-(F109-Pad2) (its old number) -> Net-(F502-Pad2)
- F503 pad 1: Net-(F110-Pad1) (its old number) -> Net-(F203-Pad2)
- F503 pad 2: Net-(F110-Pad2) (its old number) -> Net-(F503-Pad2)
- F504 pad 1: Net-(F111-Pad1) (its old number) -> Net-(F204-Pad2)
- F504 pad 2: Net-(F111-Pad2) (its old number) -> Net-(F504-Pad2)
- F505 pad 1: Net-(F112-Pad1) (its old number) -> Net-(F205-Pad2)
- F505 pad 2: Net-(F112-Pad2) -> Net-(F505-Pad2)
- F506 pad 1: Net-(F113-Pad1) (its old number) -> Net-(F206-Pad2)
- F506 pad 2: Net-(F113-Pad2) -> Net-(F506-Pad2)
- F507 pad 1: Net-(F114-Pad1) (its old number) -> Net-(F207-Pad2)
- F507 pad 2: Net-(F114-Pad2) -> Net-(F507-Pad2)
- F508 pad 1: Net-(F115-Pad1) (its old number) -> Net-(F208-Pad2)
- F508 pad 2: Net-(F115-Pad2) -> Net-(F508-Pad2)
- F509 pad 1: Net-(F116-Pad1) (its old number) -> Net-(F209-Pad2)
- F509 pad 2: Net-(F116-Pad2) -> Net-(F509-Pad2)
- F510 pad 1: Net-(F117-Pad1) (its old number) -> Net-(F210-Pad2)
- F510 pad 2: Net-(F117-Pad2) -> Net-(F510-Pad2)
- F511 pad 1: Net-(F118-Pad1) (its old number) -> Net-(F211-Pad2)
- F511 pad 2: Net-(F118-Pad2) -> Net-(F511-Pad2)
- F512 pad 2: Net-(F140-Pad2) -> Net-(F512-Pad2)
- F513 pad 2: Net-(F141-Pad2) -> Net-(F513-Pad2)
- F514 pad 2: Net-(F142-Pad2) -> Net-(F514-Pad2)
- F515 pad 2: Net-(F143-Pad2) -> Net-(F515-Pad2)
- F516 pad 2: Net-(F144-Pad2) -> Net-(F516-Pad2)
- F517 pad 2: Net-(F145-Pad2) -> Net-(F517-Pad2)
- F518 pad 2: Net-(F146-Pad2) -> Net-(F518-Pad2)
- F519 pad 2: Net-(F147-Pad2) -> Net-(F519-Pad2)
- F520 pad 2: Net-(F148-Pad2) -> Net-(F520-Pad2)
- F521 pad 2: Net-(F149-Pad2) -> Net-(F521-Pad2)
- F522 pad 1: Net-(F171-Pad1) -> Net-(F222-Pad2)
- F522 pad 2: Net-(F171-Pad2) -> Net-(F522-Pad2)
- F523 pad 1: Net-(F172-Pad1) -> Net-(F223-Pad2)
- F523 pad 2: Net-(F172-Pad2) -> Net-(F523-Pad2)
- F524 pad 1: Net-(F173-Pad1) -> Net-(F224-Pad2)
- F524 pad 2: Net-(F173-Pad2) -> Net-(F524-Pad2)
- F525 pad 1: Net-(F174-Pad1) -> Net-(F225-Pad2)
- F525 pad 2: Net-(F174-Pad2) -> Net-(F525-Pad2)
- F526 pad 1: Net-(F175-Pad1) -> Net-(F226-Pad2)
- F526 pad 2: Net-(F175-Pad2) -> Net-(F526-Pad2)
- F527 pad 1: Net-(F176-Pad1) -> Net-(F227-Pad2)
- F527 pad 2: Net-(F176-Pad2) -> Net-(F527-Pad2)
- F528 pad 1: Net-(F177-Pad1) -> Net-(F228-Pad2)
- F528 pad 2: Net-(F177-Pad2) -> Net-(F528-Pad2)
- F529 pad 1: Net-(F178-Pad1) -> Net-(F229-Pad2)
- F529 pad 2: Net-(F178-Pad2) -> Net-(F529-Pad2)
- F530 pad 1: Net-(F179-Pad1) -> Net-(F230-Pad2)
- F530 pad 2: Net-(F179-Pad2) -> Net-(F530-Pad2)
- F531 pad 1: Net-(F180-Pad1) -> Net-(F231-Pad2)
- F531 pad 2: Net-(F180-Pad2) -> Net-(F531-Pad2)
- F532 pad 1: Net-(F181-Pad1) -> Net-(F232-Pad2)
- F532 pad 2: Net-(F181-Pad2) -> Net-(F532-Pad2)
- F601 pad 1: Net-(F119-Pad1) -> Net-(F301-Pad2)
- F601 pad 2: Net-(F119-Pad2) -> Net-(F601-Pad2)
- F602 pad 1: Net-(F120-Pad1) -> Net-(F302-Pad2)
- F602 pad 2: Net-(F120-Pad2) -> Net-(F602-Pad2)
- F603 pad 1: Net-(F121-Pad1) -> Net-(F303-Pad2)
- F603 pad 2: Net-(F121-Pad2) -> Net-(F603-Pad2)
- F604 pad 1: Net-(F122-Pad1) -> Net-(F304-Pad2)
- F604 pad 2: Net-(F122-Pad2) -> Net-(F604-Pad2)
- F605 pad 1: Net-(F123-Pad1) -> Net-(F305-Pad2)
- F605 pad 2: Net-(F123-Pad2) -> Net-(F605-Pad2)
- F606 pad 1: Net-(F124-Pad1) -> Net-(F306-Pad2)
- F606 pad 2: Net-(F124-Pad2) -> Net-(F606-Pad2)
- F607 pad 1: Net-(F125-Pad1) -> Net-(F307-Pad2)
- F607 pad 2: Net-(F125-Pad2) -> Net-(F607-Pad2)
- F608 pad 1: Net-(F126-Pad1) -> Net-(F308-Pad2)
- F608 pad 2: Net-(F126-Pad2) -> Net-(F608-Pad2)
- F609 pad 1: Net-(F127-Pad1) -> Net-(F309-Pad2)
- F609 pad 2: Net-(F127-Pad2) -> Net-(F609-Pad2)
- F610 pad 1: Net-(F128-Pad1) -> Net-(F310-Pad2)
- F610 pad 2: Net-(F128-Pad2) -> Net-(F610-Pad2)
- F611 pad 1: Net-(F129-Pad1) -> Net-(F311-Pad2)
- F611 pad 2: Net-(F129-Pad2) -> Net-(F611-Pad2)
- F612 pad 1: Net-(F150-Pad1) -> Net-(F312-Pad2)
- F612 pad 2: Net-(F150-Pad2) -> Net-(F612-Pad2)
- F613 pad 1: Net-(F151-Pad1) -> Net-(F313-Pad2)
- F613 pad 2: Net-(F151-Pad2) -> Net-(F613-Pad2)
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